Commit message: add prismatic joints to model

File: meshes/environment.urdf (robot description, URDF)
Before this commit: robot cartesian_envrionment, 4 links, 3 joints
Links:
- added link prismatic_output
- added link start_pose_offset_link
- added link x_to_y
- added link y_to_z
Joints:
- removed joint table_to_gripper
- added joint prismatic_to_gripper: type fixed, parent prismatic_output, child gripper_base, origin xyz=0 0 0.560 rpy=0 1.47 0
- added joint start_pose_offset_fixed_joint: type fixed, parent base_link, child start_pose_offset_link, origin xyz=0 0 0
- added joint table_to_gripper_x: type prismatic, parent base_link, child x_to_y, origin xyz=0 0 0 rpy=0 0 0, limit lower=-0.5 upper=0.5 effort=1000 velocity=0.1
- added joint table_to_gripper_y: type prismatic, parent x_to_y, child y_to_z, origin xyz=0 0 0 rpy=0 0 1.47, limit lower=-0.5 upper=0.5 effort=1000 velocity=0.1
- added joint table_to_gripper_z: type prismatic, parent y_to_z, child prismatic_output, origin xyz=0 0 0 rpy=0 -1.47 0 , limit lower=-0.5 upper=0.5 effort=1000 velocity=0.1
- joint gripper_to_finger1: origin xyz=0.048 0 -0.185 rpy=0 0 0 -> xyz=0.048 0 -0.125 rpy=0 0 0
- joint gripper_to_finger2: origin xyz=-0.048 0 -0.185 rpy=0 0 0 -> xyz=-0.048 0 -0.125 rpy=0 0 0
