Commit message: urdf converted to xrdf

File: urdf/environment.urdf (robot description, URDF)
Before this commit: robot cartesian_envrionment, 8 links, 7 joints
Joints:
- joint prismatic_to_gripper: origin xyz=0 0 0.560 rpy=0 1.47 0 -> xyz=0 0 0.560 rpy=0 1.57079632679 0
- joint table_to_gripper_y: origin xyz=0 0 0 rpy=0 0 1.47 -> xyz=0 0 0 rpy=0 0 1.57079632679
- joint table_to_gripper_z: origin xyz=0 0 0 rpy=0 -1.47 0  -> xyz=0 0 0 rpy=0 -1.57079632679 0 

Commit message: general implementation of pybullet now working

File: urdf/environment.urdf (robot description, URDF)
Before this commit: robot cartesian_envrionment, 8 links, 7 joints
Links:
- removed link finger1
- removed link finger2
- added link finger_left; collision mesh filename=./meshes/gripper_finger.stl; visual mesh filename=./meshes/gripper_finger.stl
- added link finger_right; collision mesh filename=./meshes/gripper_finger.stl; visual mesh filename=./meshes/gripper_finger.stl
- link base_link: geometry collision mesh filename=./meshes/table.stl; visual mesh filename=./meshes/table.stl
- link gripper_base: geometry collision mesh filename=./meshes/gripper_base.stl; visual mesh filename=./meshes/gripper_base.stl
Joints:
- removed joint gripper_to_finger1
- removed joint gripper_to_finger2
- added joint gripper_to_finger_left: type fixed, parent gripper_base, child finger_left, origin xyz=0.048 0 -0.125 rpy=0 0 0
- added joint gripper_to_finger_right: type fixed, parent gripper_base, child finger_right, origin xyz=-0.048 0 -0.125 rpy=0 0 0
