Commit message: major restructure

File: simple_grasping/resources/environment.xacro (robot description, xacro)
@@ -56,4 +56,8 @@
     </joint>
     <link name="gripper_base">
+        <intertial>
+            <origin rpy="0 0 0" xyz="-0.0900 -0.0001 -0.0017" />
+            <mass value="1.5175" />
+        </intertial>
         <visual>
             <geometry>
@@ -78,4 +82,8 @@
     </joint>
     <link name="finger_left">
+        <intertial>
+            <origin rpy="0 0 0" xyz="-0.01 0 0" />
+            <mass value="0.0798" />
+        </intertial>
         <visual>
             <geometry>
@@ -90,4 +98,8 @@
     </link>
     <link name="finger_right">
+        <intertial>
+            <origin rpy="0 0 0" xyz="-0.01 0 0" />
+            <mass value="0.0798" />
+        </intertial>
         <visual>
             <geometry>
