Commit message: tweaks for calls, still some bugfixing needed

File: simple_grasping/resources/simplefetch.xacro (robot description, xacro)
@@ -4,4 +4,8 @@
 <!--robot name="cartesian_envrionment"-->
     <link name="base_link">
+        <intertial>
+            <origin rpy="0 0 0" xyz="0 0 0" />
+            <mass value="0" />
+        </intertial>
         <visual>
             <geometry>
@@ -21,4 +25,8 @@
     </joint>
     <link name="start_pose_offset_link">
+        <intertial>
+            <origin rpy="0 0 0" xyz="0 0 0" />
+            <mass value="0" />
+        </intertial>
         <origin xyz="0 0 0" rpy="0 0 0" />
     </link>
@@ -30,4 +38,8 @@
     </joint>
     <link name="x_to_y">
+        <intertial>
+            <origin rpy="0 0 0" xyz="0 0 0" />
+            <mass value="0" />
+        </intertial>
         <origin xyz="0 0 0" rpy="0 0 0"/>
     </link>
@@ -39,4 +51,8 @@
     </joint>
     <link name="y_to_z">
+        <intertial>
+            <origin rpy="0 0 0" xyz="0 0 0" />
+            <mass value="0" />
+        </intertial>
         <origin xyz="0 0 0" rpy="0 0 0"/>
     </link>
@@ -48,4 +64,8 @@
     </joint>
     <link name="prismatic_output">
+        <intertial>
+            <origin rpy="0 0 0" xyz="0 0 0" />
+            <mass value="0" />
+        </intertial>
         <origin xyz="0 0 0" rpy="0 0 0"/>
     </link>

Commit message: fix urdf-based warnings

File: simple_grasping/resources/simplefetch.xacro (robot description, xacro)
@@ -14,4 +14,9 @@
             </geometry>
         </collision>
+        <inertial>
+            <origin rpy="0 0 0" xyz="0 0 0" />
+            <mass value="0" />
+            <inertia ixx="0" ixy="0" iyy="0" izz="0"/>
+        </inertial>
     </link>
     <joint name="start_pose_offset_fixed_joint" type="fixed">
@@ -19,7 +24,13 @@
         <child link="start_pose_offset_link" />
         <origin xyz="0 0 0" />
+        <axis xyz="1 0 0" />
     </joint>
     <link name="start_pose_offset_link">
         <origin xyz="0 0 0" rpy="0 0 0" />
+        <inertial>
+            <origin rpy="0 0 0" xyz="0 0 0" />
+            <mass value="0" />
+            <inertia ixx="0" ixy="0" iyy="0" izz="0"/>
+        </inertial>
     </link>
     <joint name="table_to_gripper_x" type="prismatic">
@@ -28,7 +39,13 @@
         <origin xyz="0 0 0" rpy="0 0 0" />
         <limit effort="1000" lower="-0.5" upper="0.5" velocity="0.1" />
+        <axis xyz="1 0 0" />
     </joint>
     <link name="x_to_y">
         <origin xyz="0 0 0" rpy="0 0 0"/>
+        <inertial>
+            <origin rpy="0 0 0" xyz="0 0 0" />
+            <mass value="0" />
+            <inertia ixx="0" ixy="0" iyy="0" izz="0"/>
+        </inertial>
     </link>
     <joint name="table_to_gripper_y" type="prismatic">
@@ -37,7 +54,13 @@
         <origin xyz="0 0 0" rpy="0 0 ${pi/2}" />
         <limit effort="1000" lower="-0.5" upper="0.5" velocity="0.1" />
+        <axis xyz="1 0 0" />
     </joint>
     <link name="y_to_z">
         <origin xyz="0 0 0" rpy="0 0 0"/>
+        <inertial>
+            <origin rpy="0 0 0" xyz="0 0 0" />
+            <mass value="0" />
+            <inertia ixx="0" ixy="0" iyy="0" izz="0"/>
+        </inertial>
     </link>
     <joint name="table_to_gripper_z" type="prismatic">
@@ -46,7 +69,13 @@
         <origin xyz="0 0 0" rpy="0 -${pi/2} 0 " />
         <limit effort="1000" lower="-0.5" upper="0.5" velocity="0.1" />
+        <axis xyz="1 0 0" />
     </joint>
     <link name="prismatic_output">
         <origin xyz="0 0 0" rpy="0 0 0"/>
+        <inertial>
+            <origin rpy="0 0 0" xyz="0 0 0" />
+            <mass value="0" />
+            <inertia ixx="0" ixy="0" iyy="0" izz="0"/>
+        </inertial>
     </link>
     <joint name="prismatic_to_gripper" type="fixed">
@@ -54,4 +83,5 @@
         <child link="gripper_base" />
         <origin xyz="0.560 -0.25 -0.25" rpy="0 ${pi/2} 0" />
+        <axis xyz="1 0 0" />
     </joint>
     <link name="gripper_base">
@@ -77,4 +107,5 @@
         <child link="finger_left" />
         <origin xyz="0.048 0 -0.125" rpy="0 0 ${pi/2}" />
+        <axis xyz="1 0 0" />
     </joint>
     <joint name="gripper_to_finger_right" type="prismatic">
@@ -83,4 +114,5 @@
         <child link="finger_right" />
         <origin xyz="-0.048 0 -0.125" rpy="0 0 ${pi/2}" />
+        <axis xyz="1 0 0" />
     </joint>
     <link name="finger_left">
