Commit message: medium and small blocks as xacros as well

File: simple_grasping/resources/medium_block.urdf (robot description, URDF)
Before this commit: robot small_block, 4 links, 4 joints
Links:
- removed link inertial_link
- added link block, mass 1; collision box size=0.06 0.06 0.06; visual box size=0.06 0.06 0.06
- link base_link: geometry 
Joints:
- removed joint fixed_inertial_joint
- joint base_to_cube_z: child prismatic_output -> block

File: simple_grasping/resources/medium_block.xacro (robot description, xacro)
@@ -12,15 +12,4 @@
     <link name="base_link">
         <origin rpy="0 0 0" xyz="0 0 0"/>
-        <visual>
-            <geometry>
-                <box size="0.06 0.06 0.06"/>
-            </geometry>
-            <material name="white" />
-        </visual>
-        <collision>
-            <geometry>
-                <box size="0.06 0.06 0.06"/>
-            </geometry>
-        </collision>
         <inertial>
             <origin rpy="0 0 0" xyz="0 0 0"/>
@@ -61,15 +50,21 @@
     <joint name="base_to_cube_z" type="prismatic">
         <parent link="y_to_z" />
-        <child link="prismatic_output" />
+        <child link="block" />
         <origin xyz="0 0 0" rpy="0 -${pi/2} 0 " />
         <limit effort="1000" lower="-50" upper="50" velocity="10" />
         <axis xyz="1 0 0" />
     </joint>
-    <!-- workaround for the fact that base links don't have mass/inertia -->
-    <joint name="fixed_inertial_joint" type="fixed">
-        <child link="inertial_link" />
-        <parent link="base_link" />
-    </joint>
-    <link name="inertial_link">
+    <link name="block">
+        <visual>
+            <geometry>
+                <box size="0.06 0.06 0.06"/>
+            </geometry>
+            <material name="white" />
+        </visual>
+        <collision>
+            <geometry>
+                <box size="0.06 0.06 0.06"/>
+            </geometry>
+        </collision>
         <inertial>
           <origin rpy="0 0 0" xyz="0 0 0"/>

File: simple_grasping/resources/small_block.urdf (robot description, URDF)
Before this commit: robot small_block, 4 links, 4 joints
Links:
- removed link inertial_link
- added link block, mass 1; collision box size=0.04 0.04 0.04; visual box size=0.04 0.04 0.04
- link base_link: geometry 
Joints:
- removed joint fixed_inertial_joint
- joint base_to_cube_z: child prismatic_output -> block

File: simple_grasping/resources/small_block.xacro (robot description, xacro)
@@ -12,15 +12,4 @@
     <link name="base_link">
         <origin rpy="0 0 0" xyz="0 0 0"/>
-        <visual>
-            <geometry>
-                <box size="0.04 0.04 0.04"/>
-            </geometry>
-            <material name="white" />
-        </visual>
-        <collision>
-            <geometry>
-                <box size="0.04 0.04 0.04"/>
-            </geometry>
-        </collision>
         <inertial>
             <origin rpy="0 0 0" xyz="0 0 0"/>
@@ -61,15 +50,21 @@
     <joint name="base_to_cube_z" type="prismatic">
         <parent link="y_to_z" />
-        <child link="prismatic_output" />
+        <child link="block" />
         <origin xyz="0 0 0" rpy="0 -${pi/2} 0 " />
         <limit effort="1000" lower="-50" upper="50" velocity="10" />
         <axis xyz="1 0 0" />
     </joint>
-    <!-- workaround for the fact that base links don't have mass/inertia -->
-    <joint name="fixed_inertial_joint" type="fixed">
-        <child link="inertial_link" />
-        <parent link="base_link" />
-    </joint>
-    <link name="inertial_link">
+    <link name="block">
+        <visual>
+            <geometry>
+                <box size="0.04 0.04 0.04"/>
+            </geometry>
+            <material name="white" />
+        </visual>
+        <collision>
+            <geometry>
+                <box size="0.04 0.04 0.04"/>
+            </geometry>
+        </collision>
         <inertial>
           <origin rpy="0 0 0" xyz="0 0 0"/>
