Commit message: urdf changes, add meshes, sequential agent

File: simple_grasping/resources/large_block.urdf (robot description, URDF)
Before this commit: robot small_block, 2 links, 1 joints
Links:
- link base_link: mass None -> 0; geometry collision mesh filename=file:///home/cst/code/pybullet_simplified_fetch/simple_gras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; visual mesh filename=file:///home/cst/code/pybullet_simplified_fetch/simple_gras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

File: simple_grasping/resources/medium_block.urdf (robot description, URDF)
Before this commit: robot small_block, 2 links, 1 joints
Links:
- link base_link: mass None -> 0; geometry collision mesh filename=file:///home/cst/code/pybullet_simplified_fetch/simple_gras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; visual mesh filename=file:///home/cst/code/pybullet_simplified_fetch/simple_gras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

File: simple_grasping/resources/simplefetch.urdf (robot description, URDF)
Before this commit: robot cartesian_envrionment, 8 links, 7 joints
Joints:
- joint prismatic_to_gripper: origin xyz=0.560 -0.25 -0.25 rpy=0 1.57079632679 0 -> xyz=0.560 0 0 rpy=0 1.57079632679 0

File: simple_grasping/resources/simplefetch.xacro (robot description, xacro)
@@ -82,5 +82,5 @@
         <parent link="prismatic_output" />
         <child link="gripper_base" />
-        <origin xyz="0.560 -0.25 -0.25" rpy="0 ${pi/2} 0" />
+        <origin xyz="0.560 0 0" rpy="0 ${pi/2} 0" />
         <axis xyz="1 0 0" />
     </joint>

File: simple_grasping/resources/small_block.urdf (robot description, URDF)
Before this commit: robot small_block, 2 links, 1 joints
Links:
- link base_link: mass None -> 0; geometry collision mesh filename=file:///home/cst/code/pybullet_simplified_fetch/simple_gras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; visual mesh filename=file:///home/cst/code/pybullet_simplified_fetch/simple_gras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

Commit message: major bugfixes: velocity movement, block placement, BlockObject

File: simple_grasping/resources/large_block.urdf (robot description, URDF)
Before this commit: robot small_block, 2 links, 1 joints
Links:
- link base_link: geometry collision box size=0.08 0.08 0.08; visual box size=0.08 0.08 0.08

File: simple_grasping/resources/large_block.xacro (robot description, xacro)
@@ -14,5 +14,5 @@
         <visual>
             <geometry>
-                <mesh filename="file://$(cwd)/meshes/80mm.stl"/>
+                <box size="0.08 0.08 0.08"/>
             </geometry>
             <material name="white" />
@@ -20,5 +20,5 @@
         <collision>
             <geometry>
-                <mesh filename="file://$(cwd)/meshes/80mm.stl"/>
+                <box size="0.08 0.08 0.08"/>
             </geometry>
         </collision>

File: simple_grasping/resources/medium_block.urdf (robot description, URDF)
Before this commit: robot small_block, 2 links, 1 joints
Links:
- link base_link: geometry collision box size=0.06 0.06 0.06; visual box size=0.06 0.06 0.06

File: simple_grasping/resources/medium_block.xacro (robot description, xacro)
@@ -14,5 +14,5 @@
         <visual>
             <geometry>
-                <mesh filename="file://$(cwd)/meshes/60mm.stl"/>
+                <box size="0.06 0.06 0.06"/>
             </geometry>
             <material name="white" />
@@ -20,5 +20,5 @@
         <collision>
             <geometry>
-                <mesh filename="file://$(cwd)/meshes/60mm.stl"/>
+                <box size="0.06 0.06 0.06"/>
             </geometry>
         </collision>

File: simple_grasping/resources/simplefetch.urdf (robot description, URDF)
Before this commit: robot cartesian_envrionment, 8 links, 7 joints
Joints:
- joint table_to_gripper_x: limit lower=-0.5 upper=0.5 effort=1000 velocity=0.1 -> lower=-50 upper=50 effort=1000 velocity=10
- joint table_to_gripper_y: limit lower=-0.5 upper=0.5 effort=1000 velocity=0.1 -> lower=-50 upper=50 effort=1000 velocity=10
- joint table_to_gripper_z: limit lower=-0.5 upper=0.5 effort=1000 velocity=0.1 -> lower=-50 upper=50 effort=1000 velocity=10

File: simple_grasping/resources/simplefetch.xacro (robot description, xacro)
@@ -38,5 +38,5 @@
         <child link="x_to_y" />
         <origin xyz="0 0 0" rpy="0 0 0" />
-        <limit effort="1000" lower="-0.5" upper="0.5" velocity="0.1" />
+        <limit effort="1000" lower="-50" upper="50" velocity="10" />
         <axis xyz="1 0 0" />
     </joint>
@@ -53,5 +53,5 @@
         <child link="y_to_z" />
         <origin xyz="0 0 0" rpy="0 0 ${pi/2}" />
-        <limit effort="1000" lower="-0.5" upper="0.5" velocity="0.1" />
+        <limit effort="1000" lower="-50" upper="50" velocity="10" />
         <axis xyz="1 0 0" />
     </joint>
@@ -68,5 +68,5 @@
         <child link="prismatic_output" />
         <origin xyz="0 0 0" rpy="0 -${pi/2} 0 " />
-        <limit effort="1000" lower="-0.5" upper="0.5" velocity="0.1" />
+        <limit effort="1000" lower="-50" upper="50" velocity="10" />
         <axis xyz="1 0 0" />
     </joint>

File: simple_grasping/resources/small_block.urdf (robot description, URDF)
Before this commit: robot small_block, 2 links, 1 joints
Links:
- link base_link: geometry collision box size=0.04 0.04 0.04; visual box size=0.04 0.04 0.04

File: simple_grasping/resources/small_block.xacro (robot description, xacro)
@@ -14,5 +14,5 @@
         <visual>
             <geometry>
-                <mesh filename="file://$(cwd)/meshes/40mm.stl"/>
+                <box size="0.04 0.04 0.04"/>
             </geometry>
             <material name="white" />
@@ -20,5 +20,5 @@
         <collision>
             <geometry>
-                <mesh filename="file://$(cwd)/meshes/40mm.stl"/>
+                <box size="0.04 0.04 0.04"/>
             </geometry>
         </collision>

Commit message: update models to allow movement

File: simple_grasping/resources/large_block.urdf (robot description, URDF)
Before this commit: robot small_block, 2 links, 1 joints
Links:
- added link x_to_y, mass 0
- added link y_to_z, mass 0
Joints:
- added joint base_to_cube_x: type prismatic, parent base_link, child x_to_y, origin xyz=0 0 0 rpy=0 0 0, axis 1 0 0, limit lower=-50 upper=50 effort=1000 velocity=10
- added joint base_to_cube_y: type prismatic, parent x_to_y, child y_to_z, origin xyz=0 0 0 rpy=0 0 1.57079632679, axis 1 0 0, limit lower=-50 upper=50 effort=1000 velocity=10
- added joint base_to_cube_z: type prismatic, parent y_to_z, child prismatic_output, origin xyz=0 0 0 rpy=0 -1.57079632679 0 , axis 1 0 0, limit lower=-50 upper=50 effort=1000 velocity=10

File: simple_grasping/resources/large_block.xacro (robot description, xacro)
@@ -29,4 +29,41 @@
         </inertial>
     </link>
+    <joint name="base_to_cube_x" type="prismatic">
+        <parent link="base_link" />
+        <child link="x_to_y" />
+        <origin xyz="0 0 0" rpy="0 0 0" />
+        <limit effort="1000" lower="-50" upper="50" velocity="10" />
+        <axis xyz="1 0 0" />
+    </joint>
+    <link name="x_to_y">
+        <origin xyz="0 0 0" rpy="0 0 0"/>
+        <inertial>
+            <origin rpy="0 0 0" xyz="0 0 0" />
+            <mass value="0" />
+            <inertia ixx="0" ixy="0" ixz="0" iyy="0" iyz="0" izz="0"/>
+        </inertial>
+    </link>
+    <joint name="base_to_cube_y" type="prismatic">
+        <parent link="x_to_y" />
+        <child link="y_to_z" />
+        <origin xyz="0 0 0" rpy="0 0 ${pi/2}" />
+        <limit effort="1000" lower="-50" upper="50" velocity="10" />
+        <axis xyz="1 0 0" />
+    </joint>
+    <link name="y_to_z">
+        <origin xyz="0 0 0" rpy="0 0 0"/>
+        <inertial>
+            <origin rpy="0 0 0" xyz="0 0 0" />
+            <mass value="0" />
+            <inertia ixx="0" ixy="0" ixz="0" iyy="0" iyz="0" izz="0"/>
+        </inertial>
+    </link>
+    <joint name="base_to_cube_z" type="prismatic">
+        <parent link="y_to_z" />
+        <child link="prismatic_output" />
+        <origin xyz="0 0 0" rpy="0 -${pi/2} 0 " />
+        <limit effort="1000" lower="-50" upper="50" velocity="10" />
+        <axis xyz="1 0 0" />
+    </joint>
     <!-- workaround for the fact that base links don't have mass/inertia -->
     <joint name="fixed_inertial_joint" type="fixed">

File: simple_grasping/resources/medium_block.urdf (robot description, URDF)
Before this commit: robot small_block, 2 links, 1 joints
Links:
- added link x_to_y, mass 0
- added link y_to_z, mass 0
Joints:
- added joint base_to_cube_x: type prismatic, parent base_link, child x_to_y, origin xyz=0 0 0 rpy=0 0 0, axis 1 0 0, limit lower=-50 upper=50 effort=1000 velocity=10
- added joint base_to_cube_y: type prismatic, parent x_to_y, child y_to_z, origin xyz=0 0 0 rpy=0 0 1.57079632679, axis 1 0 0, limit lower=-50 upper=50 effort=1000 velocity=10
- added joint base_to_cube_z: type prismatic, parent y_to_z, child prismatic_output, origin xyz=0 0 0 rpy=0 -1.57079632679 0 , axis 1 0 0, limit lower=-50 upper=50 effort=1000 velocity=10

File: simple_grasping/resources/medium_block.xacro (robot description, xacro)
@@ -29,4 +29,41 @@
         </inertial>
     </link>
+    <joint name="base_to_cube_x" type="prismatic">
+        <parent link="base_link" />
+        <child link="x_to_y" />
+        <origin xyz="0 0 0" rpy="0 0 0" />
+        <limit effort="1000" lower="-50" upper="50" velocity="10" />
+        <axis xyz="1 0 0" />
+    </joint>
+    <link name="x_to_y">
+        <origin xyz="0 0 0" rpy="0 0 0"/>
+        <inertial>
+            <origin rpy="0 0 0" xyz="0 0 0" />
+            <mass value="0" />
+            <inertia ixx="0" ixy="0" ixz="0" iyy="0" iyz="0" izz="0"/>
+        </inertial>
+    </link>
+    <joint name="base_to_cube_y" type="prismatic">
+        <parent link="x_to_y" />
+        <child link="y_to_z" />
+        <origin xyz="0 0 0" rpy="0 0 ${pi/2}" />
+        <limit effort="1000" lower="-50" upper="50" velocity="10" />
+        <axis xyz="1 0 0" />
+    </joint>
+    <link name="y_to_z">
+        <origin xyz="0 0 0" rpy="0 0 0"/>
+        <inertial>
+            <origin rpy="0 0 0" xyz="0 0 0" />
+            <mass value="0" />
+            <inertia ixx="0" ixy="0" ixz="0" iyy="0" iyz="0" izz="0"/>
+        </inertial>
+    </link>
+    <joint name="base_to_cube_z" type="prismatic">
+        <parent link="y_to_z" />
+        <child link="prismatic_output" />
+        <origin xyz="0 0 0" rpy="0 -${pi/2} 0 " />
+        <limit effort="1000" lower="-50" upper="50" velocity="10" />
+        <axis xyz="1 0 0" />
+    </joint>
     <!-- workaround for the fact that base links don't have mass/inertia -->
     <joint name="fixed_inertial_joint" type="fixed">

File: simple_grasping/resources/simplefetch.urdf (robot description, URDF)
Before this commit: robot cartesian_envrionment, 8 links, 7 joints
Joints:
- joint prismatic_to_gripper: origin xyz=0.550 0 0 rpy=0 1.57079632679 0 -> xyz=0.55 0.0 0.0 rpy=0 1.57079632679 0

File: simple_grasping/resources/simplefetch.xacro (robot description, xacro)
@@ -82,10 +82,10 @@
         <parent link="prismatic_output" />
         <child link="gripper_base" />
-        <origin xyz="0.550 0 0" rpy="0 ${pi/2} 0" />
+        <origin xyz="0.55 0.0 0.0" rpy="0 ${pi/2} 0" />
         <axis xyz="1 0 0" />
     </joint>
     <link name="gripper_base">
         <inertial>
-            <origin rpy="0 0 0" xyz="-0.0900 -0.0001 -0.0017" />
+            <origin rpy="0 0 0" xyz="0.000 -0.06 -0.0017"/>
             <mass value="1.5175" />
             <inertia ixx="0.0013" ixy="-0.0" ixz="0.0" iyy="0.0019" iyz="-0.0" izz="0.0024" />

File: simple_grasping/resources/small_block.urdf (robot description, URDF)
Before this commit: robot small_block, 2 links, 1 joints
Links:
- added link x_to_y, mass 0
- added link y_to_z, mass 0
Joints:
- added joint base_to_cube_x: type prismatic, parent base_link, child x_to_y, origin xyz=0 0 0 rpy=0 0 0, axis 1 0 0, limit lower=-50 upper=50 effort=1000 velocity=10
- added joint base_to_cube_y: type prismatic, parent x_to_y, child y_to_z, origin xyz=0 0 0 rpy=0 0 1.57079632679, axis 1 0 0, limit lower=-50 upper=50 effort=1000 velocity=10
- added joint base_to_cube_z: type prismatic, parent y_to_z, child prismatic_output, origin xyz=0 0 0 rpy=0 -1.57079632679 0 , axis 1 0 0, limit lower=-50 upper=50 effort=1000 velocity=10

File: simple_grasping/resources/small_block.xacro (robot description, xacro)
@@ -29,4 +29,41 @@
         </inertial>
     </link>
+    <joint name="base_to_cube_x" type="prismatic">
+        <parent link="base_link" />
+        <child link="x_to_y" />
+        <origin xyz="0 0 0" rpy="0 0 0" />
+        <limit effort="1000" lower="-50" upper="50" velocity="10" />
+        <axis xyz="1 0 0" />
+    </joint>
+    <link name="x_to_y">
+        <origin xyz="0 0 0" rpy="0 0 0"/>
+        <inertial>
+            <origin rpy="0 0 0" xyz="0 0 0" />
+            <mass value="0" />
+            <inertia ixx="0" ixy="0" ixz="0" iyy="0" iyz="0" izz="0"/>
+        </inertial>
+    </link>
+    <joint name="base_to_cube_y" type="prismatic">
+        <parent link="x_to_y" />
+        <child link="y_to_z" />
+        <origin xyz="0 0 0" rpy="0 0 ${pi/2}" />
+        <limit effort="1000" lower="-50" upper="50" velocity="10" />
+        <axis xyz="1 0 0" />
+    </joint>
+    <link name="y_to_z">
+        <origin xyz="0 0 0" rpy="0 0 0"/>
+        <inertial>
+            <origin rpy="0 0 0" xyz="0 0 0" />
+            <mass value="0" />
+            <inertia ixx="0" ixy="0" ixz="0" iyy="0" iyz="0" izz="0"/>
+        </inertial>
+    </link>
+    <joint name="base_to_cube_z" type="prismatic">
+        <parent link="y_to_z" />
+        <child link="prismatic_output" />
+        <origin xyz="0 0 0" rpy="0 -${pi/2} 0 " />
+        <limit effort="1000" lower="-50" upper="50" velocity="10" />
+        <axis xyz="1 0 0" />
+    </joint>
     <!-- workaround for the fact that base links don't have mass/inertia -->
     <joint name="fixed_inertial_joint" type="fixed">

Commit message: add large block as prismatic object

File: simple_grasping/resources/large_block.urdf (robot description, URDF)
Before this commit: robot small_block, 4 links, 4 joints
Links:
- removed link inertial_link
- added link block, mass 1; collision box size=0.08 0.08 0.08; visual box size=0.08 0.08 0.08
- link base_link: geometry 
Joints:
- removed joint fixed_inertial_joint
- joint base_to_cube_z: child prismatic_output -> block

File: simple_grasping/resources/large_block.xacro (robot description, xacro)
@@ -12,15 +12,4 @@
     <link name="base_link">
         <origin rpy="0 0 0" xyz="0 0 0"/>
-        <visual>
-            <geometry>
-                <box size="0.08 0.08 0.08"/>
-            </geometry>
-            <material name="white" />
-        </visual>
-        <collision>
-            <geometry>
-                <box size="0.08 0.08 0.08"/>
-            </geometry>
-        </collision>
         <inertial>
             <origin rpy="0 0 0" xyz="0 0 0"/>
@@ -61,15 +50,21 @@
     <joint name="base_to_cube_z" type="prismatic">
         <parent link="y_to_z" />
-        <child link="prismatic_output" />
+        <child link="block" />
         <origin xyz="0 0 0" rpy="0 -${pi/2} 0 " />
         <limit effort="1000" lower="-50" upper="50" velocity="10" />
         <axis xyz="1 0 0" />
     </joint>
-    <!-- workaround for the fact that base links don't have mass/inertia -->
-    <joint name="fixed_inertial_joint" type="fixed">
-        <child link="inertial_link" />
-        <parent link="base_link" />
-    </joint>
-    <link name="inertial_link">
+    <link name="block">
+        <visual>
+            <geometry>
+                <box size="0.08 0.08 0.08"/>
+            </geometry>
+            <material name="white" />
+        </visual>
+        <collision>
+            <geometry>
+                <box size="0.08 0.08 0.08"/>
+            </geometry>
+        </collision>
         <inertial>
           <origin rpy="0 0 0" xyz="0 0 0"/>

Commit message: decreasing block size to improve block spawn placement

File: simple_grasping/resources/large_block.urdf (robot description, URDF)
Before this commit: robot small_block, 4 links, 3 joints
Links:
- link block: geometry collision box size=0.06 0.06 0.06; visual box size=0.06 0.06 0.06

File: simple_grasping/resources/large_block.xacro (robot description, xacro)
@@ -58,5 +58,5 @@
         <visual>
             <geometry>
-                <box size="0.08 0.08 0.08"/>
+                <box size="0.06 0.06 0.06"/>
             </geometry>
             <material name="white" />
@@ -64,5 +64,5 @@
         <collision>
             <geometry>
-                <box size="0.08 0.08 0.08"/>
+                <box size="0.06 0.06 0.06"/>
             </geometry>
         </collision>

File: simple_grasping/resources/medium_block.urdf (robot description, URDF)
Before this commit: robot small_block, 4 links, 3 joints
Links:
- link block: geometry collision box size=0.06 0.06 0.06; visual box size=0.04 0.04 0.04

File: simple_grasping/resources/medium_block.xacro (robot description, xacro)
@@ -58,5 +58,5 @@
         <visual>
             <geometry>
-                <box size="0.06 0.06 0.06"/>
+                <box size="0.04 0.04 0.04"/>
             </geometry>
             <material name="white" />
@@ -64,5 +64,5 @@
         <collision>
             <geometry>
-                <box size="0.06 0.06 0.06"/>
+                <box size="0.04 0.04 0.04"/>
             </geometry>
         </collision>

File: simple_grasping/resources/small_block.urdf (robot description, URDF)
Before this commit: robot small_block, 4 links, 3 joints
Links:
- link block: geometry collision box size=0.02 0.02 0.02; visual box size=0.02 0.02 0.02

File: simple_grasping/resources/small_block.xacro (robot description, xacro)
@@ -58,5 +58,5 @@
         <visual>
             <geometry>
-                <box size="0.04 0.04 0.04"/>
+                <box size="0.02 0.02 0.02"/>
             </geometry>
             <material name="white" />
@@ -64,5 +64,5 @@
         <collision>
             <geometry>
-                <box size="0.04 0.04 0.04"/>
+                <box size="0.02 0.02 0.02"/>
             </geometry>
         </collision>
