Commit message: fix pathing issue

File: simple_grasping/resources/simplefetch.urdf (robot description, URDF)
Before this commit: robot cartesian_envrionment, 8 links, 7 joints
Links:
- link base_link: geometry collision mesh filename=file:///home/cst/code/pybullet_simplified_fetch/simple_gras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; visual mesh filename=file:///home/cst/code/pybullet_simplified_fetch/simple_gras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
- link finger_left: geometry collision mesh filename=file:///home/cst/code/pybullet_simplified_fetch/simple_gras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; visual mesh filename=file:///home/cst/code/pybullet_simplified_fetch/simple_gras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
- link finger_right: geometry collision mesh filename=file:///home/cst/code/pybullet_simplified_fetch/simple_gras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; visual mesh filename=file:///home/cst/code/pybullet_simplified_fetch/simple_gras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
- link gripper_base: geometry collision mesh filename=file:///home/cst/code/pybullet_simplified_fetch/simple_gras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; visual mesh filename=file:///home/cst/code/pybullet_simplified_fetch/simple_gras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

File: simple_grasping/resources/simplefetch.xacro (robot description, xacro)
@@ -6,18 +6,22 @@
         <intertial>
             <origin rpy="0 0 0" xyz="0 0 0" />
-            <mass value="0" />
+            <mass value="0.001" />
         </intertial>
         <visual>
             <geometry>
-                <mesh filename="./meshes/table.stl"/>
+                <mesh filename="file://$(cwd)/meshes/table.stl"/>
             </geometry>
         </visual>
         <collision>
             <geometry>
-                <mesh filename="./meshes/table.stl"/>
+                <mesh filename="file://$(cwd)/meshes/table.stl"/>
             </geometry>
         </collision>
     </link>
     <joint name="start_pose_offset_fixed_joint" type="fixed">
+        <intertial>
+            <origin rpy="0 0 0" xyz="0 0 0" />
+            <mass value="0.001" />
+        </intertial>
         <parent link="base_link" />
         <child link="start_pose_offset_link" />
@@ -27,9 +31,13 @@
         <intertial>
             <origin rpy="0 0 0" xyz="0 0 0" />
-            <mass value="0" />
+            <mass value="0.001" />
         </intertial>
         <origin xyz="0 0 0" rpy="0 0 0" />
     </link>
     <joint name="table_to_gripper_x" type="prismatic">
+        <intertial>
+            <origin rpy="0 0 0" xyz="0 0 0" />
+            <mass value="0.001" />
+        </intertial>
         <parent link="base_link" />
         <child link="x_to_y" />
@@ -45,4 +53,8 @@
     </link>
     <joint name="table_to_gripper_y" type="prismatic">
+        <intertial>
+            <origin rpy="0 0 0" xyz="0 0 0" />
+            <mass value="0.001" />
+        </intertial>
         <parent link="x_to_y" />
         <child link="y_to_z" />
@@ -53,9 +65,13 @@
         <intertial>
             <origin rpy="0 0 0" xyz="0 0 0" />
-            <mass value="0" />
+            <mass value="0.001" />
         </intertial>
         <origin xyz="0 0 0" rpy="0 0 0"/>
     </link>
     <joint name="table_to_gripper_z" type="prismatic">
+        <intertial>
+            <origin rpy="0 0 0" xyz="0 0 0" />
+            <mass value="0.001" />
+        </intertial>
         <parent link="y_to_z" />
         <child link="prismatic_output" />
@@ -66,9 +82,13 @@
         <intertial>
             <origin rpy="0 0 0" xyz="0 0 0" />
-            <mass value="0" />
+            <mass value="0.001" />
         </intertial>
         <origin xyz="0 0 0" rpy="0 0 0"/>
     </link>
     <joint name="prismatic_to_gripper" type="fixed">
+        <intertial>
+            <origin rpy="0 0 0" xyz="0 0 0" />
+            <mass value="0.001" />
+        </intertial>
         <parent link="prismatic_output" />
         <child link="gripper_base" />
@@ -82,14 +102,18 @@
         <visual>
             <geometry>
-                <mesh filename="./meshes/gripper_base.stl"/>
+                <mesh filename="file://$(cwd)/meshes/gripper_base.stl"/>
             </geometry>
         </visual>
         <collision>
             <geometry>
-                <mesh filename="./meshes/gripper_base.stl"/>
+                <mesh filename="file://$(cwd)/meshes/gripper_base.stl"/>
             </geometry>
         </collision>
     </link>
     <joint name="gripper_to_finger_left" type="fixed">
+        <intertial>
+            <origin rpy="0 0 0" xyz="0 0 0" />
+            <mass value="0.001" />
+        </intertial>
         <parent link="gripper_base" />
         <child link="finger_left" />
@@ -97,4 +121,8 @@
     </joint>
     <joint name="gripper_to_finger_right" type="fixed">
+        <intertial>
+            <origin rpy="0 0 0" xyz="0 0 0" />
+            <mass value="0.001" />
+        </intertial>
         <parent link="gripper_base" />
         <child link="finger_right" />
@@ -108,10 +136,10 @@
         <visual>
             <geometry>
-                <mesh filename="./meshes/gripper_finger.stl"/>
+                <mesh filename="file://$(cwd)/meshes/gripper_finger.stl"/>
             </geometry>
         </visual>
         <collision>
             <geometry>
-                <mesh filename="./meshes/gripper_finger.stl"/>
+                <mesh filename="file://$(cwd)/meshes/gripper_finger.stl"/>
             </geometry>
         </collision>
@@ -124,10 +152,10 @@
         <visual>
             <geometry>
-                <mesh filename="./meshes/gripper_finger.stl"/>
+                <mesh filename="file://$(cwd)/meshes/gripper_finger.stl"/>
             </geometry>
         </visual>
         <collision>
             <geometry>
-                <mesh filename="./meshes/gripper_finger.stl"/>
+                <mesh filename="file://$(cwd)/meshes/gripper_finger.stl"/>
             </geometry>
         </collision>

Commit message: urdf fixes

File: simple_grasping/resources/simplefetch.urdf (robot description, URDF)
Before this commit: robot cartesian_envrionment, 8 links, 7 joints
Links:
- link finger_left: mass None -> 0.0798
- link finger_right: mass None -> 0.0798
- link gripper_base: mass None -> 1.5175
Joints:
- joint gripper_to_finger_left: limit (none) -> lower=0.0 upper=-0.048 effort=1000 velocity=0.1; origin xyz=0.048 0 -0.125 rpy=0 0 0 -> xyz=0.048 0 -0.125 rpy=0 0 1.57079632679; type fixed -> prismatic
- joint gripper_to_finger_right: limit (none) -> lower=0.048 upper=0.0 effort=1000 velocity=0.1; origin xyz=-0.048 0 -0.125 rpy=0 0 0 -> xyz=-0.048 0 -0.125 rpy=0 0 1.57079632679; type fixed -> prismatic
- joint prismatic_to_gripper: origin xyz=0 0 0.560 rpy=0 1.57079632679 0 -> xyz=0.560 -0.25 -0.25 rpy=0 1.57079632679 0

File: simple_grasping/resources/simplefetch.xacro (robot description, xacro)
@@ -4,8 +4,4 @@
 <!--robot name="cartesian_envrionment"-->
     <link name="base_link">
-        <intertial>
-            <origin rpy="0 0 0" xyz="0 0 0" />
-            <mass value="0.001" />
-        </intertial>
         <visual>
             <geometry>
@@ -20,8 +16,4 @@
     </link>
     <joint name="start_pose_offset_fixed_joint" type="fixed">
-        <intertial>
-            <origin rpy="0 0 0" xyz="0 0 0" />
-            <mass value="0.001" />
-        </intertial>
         <parent link="base_link" />
         <child link="start_pose_offset_link" />
@@ -29,15 +21,7 @@
     </joint>
     <link name="start_pose_offset_link">
-        <intertial>
-            <origin rpy="0 0 0" xyz="0 0 0" />
-            <mass value="0.001" />
-        </intertial>
         <origin xyz="0 0 0" rpy="0 0 0" />
     </link>
     <joint name="table_to_gripper_x" type="prismatic">
-        <intertial>
-            <origin rpy="0 0 0" xyz="0 0 0" />
-            <mass value="0.001" />
-        </intertial>
         <parent link="base_link" />
         <child link="x_to_y" />
@@ -46,15 +30,7 @@
     </joint>
     <link name="x_to_y">
-        <intertial>
-            <origin rpy="0 0 0" xyz="0 0 0" />
-            <mass value="0" />
-        </intertial>
         <origin xyz="0 0 0" rpy="0 0 0"/>
     </link>
     <joint name="table_to_gripper_y" type="prismatic">
-        <intertial>
-            <origin rpy="0 0 0" xyz="0 0 0" />
-            <mass value="0.001" />
-        </intertial>
         <parent link="x_to_y" />
         <child link="y_to_z" />
@@ -63,15 +39,7 @@
     </joint>
     <link name="y_to_z">
-        <intertial>
-            <origin rpy="0 0 0" xyz="0 0 0" />
-            <mass value="0.001" />
-        </intertial>
         <origin xyz="0 0 0" rpy="0 0 0"/>
     </link>
     <joint name="table_to_gripper_z" type="prismatic">
-        <intertial>
-            <origin rpy="0 0 0" xyz="0 0 0" />
-            <mass value="0.001" />
-        </intertial>
         <parent link="y_to_z" />
         <child link="prismatic_output" />
@@ -80,24 +48,17 @@
     </joint>
     <link name="prismatic_output">
-        <intertial>
-            <origin rpy="0 0 0" xyz="0 0 0" />
-            <mass value="0.001" />
-        </intertial>
         <origin xyz="0 0 0" rpy="0 0 0"/>
     </link>
     <joint name="prismatic_to_gripper" type="fixed">
-        <intertial>
-            <origin rpy="0 0 0" xyz="0 0 0" />
-            <mass value="0.001" />
-        </intertial>
         <parent link="prismatic_output" />
         <child link="gripper_base" />
-        <origin xyz="0 0 0.560" rpy="0 ${pi/2} 0" />
+        <origin xyz="0.560 -0.25 -0.25" rpy="0 ${pi/2} 0" />
     </joint>
     <link name="gripper_base">
-        <intertial>
+        <inertial>
             <origin rpy="0 0 0" xyz="-0.0900 -0.0001 -0.0017" />
             <mass value="1.5175" />
-        </intertial>
+            <inertia ixx="0.0013" ixy="-0.0" ixz="0.0" iyy="0.0019" iyz="-0.0" izz="0.0024" />
+        </inertial>
         <visual>
             <geometry>
@@ -111,27 +72,22 @@
         </collision>
     </link>
-    <joint name="gripper_to_finger_left" type="fixed">
-        <intertial>
-            <origin rpy="0 0 0" xyz="0 0 0" />
-            <mass value="0.001" />
-        </intertial>
+    <joint name="gripper_to_finger_left" type="prismatic">
+        <limit effort="1000" lower="0.0" upper="-0.048" velocity="0.1" />
         <parent link="gripper_base" />
         <child link="finger_left" />
-        <origin xyz="0.048 0 -0.125" rpy="0 0 0" />
+        <origin xyz="0.048 0 -0.125" rpy="0 0 ${pi/2}" />
     </joint>
-    <joint name="gripper_to_finger_right" type="fixed">
-        <intertial>
-            <origin rpy="0 0 0" xyz="0 0 0" />
-            <mass value="0.001" />
-        </intertial>
+    <joint name="gripper_to_finger_right" type="prismatic">
+        <limit effort="1000" lower="0.048" upper="0.0" velocity="0.1" />
         <parent link="gripper_base" />
         <child link="finger_right" />
-        <origin xyz="-0.048 0 -0.125" rpy="0 0 0" />
+        <origin xyz="-0.048 0 -0.125" rpy="0 0 ${pi/2}" />
     </joint>
     <link name="finger_left">
-        <intertial>
+        <inertial>
             <origin rpy="0 0 0" xyz="-0.01 0 0" />
             <mass value="0.0798" />
-        </intertial>
+            <inertia ixx="0.002" ixy="0" ixz="0" iyy="0" iyz="0" izz="0" />
+        </inertial>
         <visual>
             <geometry>
@@ -146,8 +102,9 @@
     </link>
     <link name="finger_right">
-        <intertial>
+        <inertial>
             <origin rpy="0 0 0" xyz="-0.01 0 0" />
             <mass value="0.0798" />
-        </intertial>
+            <inertia ixx="0.002" ixy="0" ixz="0" iyy="0" iyz="0" izz="0" />
+        </inertial>
         <visual>
             <geometry>

Commit message: Actually fix

File: simple_grasping/resources/simplefetch.urdf (robot description, URDF)
Before this commit: robot cartesian_envrionment, 8 links, 7 joints
Links:
- link base_link: mass None -> 0
- link prismatic_output: mass None -> 0
- link start_pose_offset_link: mass None -> 0
- link x_to_y: mass None -> 0
- link y_to_z: mass None -> 0
Joints:
- joint gripper_to_finger_left: axis (none) -> 1 0 0
- joint gripper_to_finger_right: axis (none) -> 1 0 0
- joint prismatic_to_gripper: axis (none) -> 1 0 0
- joint start_pose_offset_fixed_joint: axis (none) -> 1 0 0
- joint table_to_gripper_x: axis (none) -> 1 0 0
- joint table_to_gripper_y: axis (none) -> 1 0 0
- joint table_to_gripper_z: axis (none) -> 1 0 0

Commit message: fix gripper axis, distance

File: simple_grasping/resources/simplefetch.urdf (robot description, URDF)
Before this commit: robot cartesian_envrionment, 8 links, 7 joints
Joints:
- joint gripper_to_finger_left: axis 1 0 0 -> 0 1 0; origin xyz=0.048 0 -0.125 rpy=0 0 1.57079632679 -> xyz=0.01 0 -0.125 rpy=0 0 1.57079632679
- joint gripper_to_finger_right: axis 1 0 0 -> 0 1 0; origin xyz=-0.048 0 -0.125 rpy=0 0 1.57079632679 -> xyz=-0.01 0 -0.125 rpy=0 0 1.57079632679

File: simple_grasping/resources/simplefetch.xacro (robot description, xacro)
@@ -17,5 +17,5 @@
             <origin rpy="0 0 0" xyz="0 0 0" />
             <mass value="0" />
-            <inertia ixx="0" ixy="0" iyy="0" izz="0"/>
+            <inertia ixx="0" ixy="0" ixz="0" iyy="0" iyz="0" izz="0"/>
         </inertial>
     </link>
@@ -31,5 +31,5 @@
             <origin rpy="0 0 0" xyz="0 0 0" />
             <mass value="0" />
-            <inertia ixx="0" ixy="0" iyy="0" izz="0"/>
+            <inertia ixx="0" ixy="0" ixz="0" iyy="0" iyz="0" izz="0"/>
         </inertial>
     </link>
@@ -46,5 +46,5 @@
             <origin rpy="0 0 0" xyz="0 0 0" />
             <mass value="0" />
-            <inertia ixx="0" ixy="0" iyy="0" izz="0"/>
+            <inertia ixx="0" ixy="0" ixz="0" iyy="0" iyz="0" izz="0"/>
         </inertial>
     </link>
@@ -61,5 +61,5 @@
             <origin rpy="0 0 0" xyz="0 0 0" />
             <mass value="0" />
-            <inertia ixx="0" ixy="0" iyy="0" izz="0"/>
+            <inertia ixx="0" ixy="0" ixz="0" iyy="0" iyz="0" izz="0"/>
         </inertial>
     </link>
@@ -76,5 +76,5 @@
             <origin rpy="0 0 0" xyz="0 0 0" />
             <mass value="0" />
-            <inertia ixx="0" ixy="0" iyy="0" izz="0"/>
+            <inertia ixx="0" ixy="0" ixz="0" iyy="0" iyz="0" izz="0"/>
         </inertial>
     </link>
@@ -106,6 +106,7 @@
         <parent link="gripper_base" />
         <child link="finger_left" />
-        <origin xyz="0.048 0 -0.125" rpy="0 0 ${pi/2}" />
-        <axis xyz="1 0 0" />
+        <origin xyz="0.01 0 -0.125" rpy="0 0 ${pi/2}" />
+        <!--origin xyz="${0.048/2} 0 -0.125" rpy="0 0 ${pi/2}" /-->
+        <axis xyz="0 1 0" />
     </joint>
     <joint name="gripper_to_finger_right" type="prismatic">
@@ -113,6 +114,7 @@
         <parent link="gripper_base" />
         <child link="finger_right" />
-        <origin xyz="-0.048 0 -0.125" rpy="0 0 ${pi/2}" />
-        <axis xyz="1 0 0" />
+        <origin xyz="-0.01 0 -0.125" rpy="0 0 ${pi/2}" />
+        <!--origin xyz="${-0.048/2} 0 -0.125" rpy="0 0 ${pi/2}" /-->
+        <axis xyz="0 1 0" />
     </joint>
     <link name="finger_left">

Commit message: mild refactor

File: simple_grasping/resources/simplefetch.urdf (robot description, URDF)
Before this commit: robot cartesian_envrionment, 8 links, 7 joints
Joints:
- joint prismatic_to_gripper: origin xyz=0.560 0 0 rpy=0 1.57079632679 0 -> xyz=0.550 0 0 rpy=0 1.57079632679 0

File: simple_grasping/resources/simplefetch.xacro (robot description, xacro)
@@ -82,5 +82,5 @@
         <parent link="prismatic_output" />
         <child link="gripper_base" />
-        <origin xyz="0.560 0 0" rpy="0 ${pi/2} 0" />
+        <origin xyz="0.550 0 0" rpy="0 ${pi/2} 0" />
         <axis xyz="1 0 0" />
     </joint>

Commit message: RL agent capabilities added

File: simple_grasping/resources/simplefetch.urdf (robot description, URDF)
Before this commit: robot cartesian_envrionment, 8 links, 7 joints
Links:
- link base_link: geometry collision mesh filename=file:///media/yash/SSHD/Robotics/Tufts/Spring_21/Prob_Rob/P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; visual mesh filename=file:///media/yash/SSHD/Robotics/Tufts/Spring_21/Prob_Rob/P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
- link finger_left: geometry collision mesh filename=file:///media/yash/SSHD/Robotics/Tufts/Spring_21/Prob_Rob/P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; visual mesh filename=file:///media/yash/SSHD/Robotics/Tufts/Spring_21/Prob_Rob/P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
- link finger_right: geometry collision mesh filename=file:///media/yash/SSHD/Robotics/Tufts/Spring_21/Prob_Rob/P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; visual mesh filename=file:///media/yash/SSHD/Robotics/Tufts/Spring_21/Prob_Rob/P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
- link gripper_base: geometry collision mesh filename=file:///media/yash/SSHD/Robotics/Tufts/Spring_21/Prob_Rob/P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; visual mesh filename=file:///media/yash/SSHD/Robotics/Tufts/Spring_21/Prob_Rob/P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
Joints:
- joint gripper_to_finger_left: origin xyz=0.01 0 -0.125 rpy=0 0 1.57079632679 -> xyz=0.01 0 -0.125 rpy=0 0 1.5707963267948966
- joint gripper_to_finger_right: origin xyz=-0.01 0 -0.125 rpy=0 0 1.57079632679 -> xyz=-0.01 0 -0.125 rpy=0 0 1.5707963267948966
- joint prismatic_to_gripper: origin xyz=0.55 0.0 0.0 rpy=0 1.57079632679 0 -> xyz=0.55 0.0 0.0 rpy=0 1.5707963267948966 0
- joint table_to_gripper_y: origin xyz=0 0 0 rpy=0 0 1.57079632679 -> xyz=0 0 0 rpy=0 0 1.5707963267948966
- joint table_to_gripper_z: origin xyz=0 0 0 rpy=0 -1.57079632679 0  -> xyz=0 0 0 rpy=0 -1.5707963267948966 0 
